Commit message: Add unit tests for GamepadUtils and control kinematics
- Implement tests for `processAnalogSticks` and `buildRelativeTeleopCommand` in GamepadUtils.
- Create a new URDF file for the Piper robot model.
- Add comprehensive tests for control kinematics in the phosphobot, including absolute and relative movement functions.
- Ensure that inverse kinematics prefers the current robot joint seed and validate the end effector index.

File: phosphobot/resources/urdf/piper/urdf/piper_legacy_local.urdf (robot description, URDF)
Before this commit: robot piper, 10 links, 9 joints
Links:
- removed link gripper_base
- link base_link: mass 1.02 -> 0.162548567403693; geometry collision mesh filename=package://piper/meshes/base_link.STL; visual mesh filename=package://piper/meshes/base_link.dae
- link link1: mass 0.71 -> 0.0978679932242825; geometry collision mesh filename=package://piper/meshes/link1.STL; visual mesh filename=package://piper/meshes/link1.dae
- link link2: mass 1.17 -> 0.290888938633388; geometry collision mesh filename=package://piper/meshes/link2.STL; visual mesh filename=package://piper/meshes/link2.dae
- link link3: mass 0.5 -> 0.290847697793211; geometry collision mesh filename=package://piper/meshes/link3.STL; visual mesh filename=package://piper/meshes/link3.dae
- link link4: mass 0.38 -> 0.127087348341362; geometry collision mesh filename=package://piper/meshes/link4.STL; visual mesh filename=package://piper/meshes/link4.dae
- link link5: mass 0.383 -> 0.144711242639457; geometry collision mesh filename=package://piper/meshes/link5.STL; visual mesh filename=package://piper/meshes/link5.dae
- link link6: mass 0.00699089613564366 -> 0.195187143240719; geometry collision mesh filename=package://piper/meshes/link6_1.STL; visual mesh filename=package://piper/meshes/link6.dae
- link link7: mass 0.025 -> 0.02648229234527; geometry collision mesh filename=package://piper/meshes/link7.STL; visual mesh filename=package://piper/meshes/link7.dae
- link link8: mass 0.025 -> 0.0264822021416248; geometry collision mesh filename=package://piper/meshes/link8.STL; visual mesh filename=package://piper/meshes/link8.dae
Joints:
- removed joint joint6_to_gripper_base
- joint joint1: limit lower=-2.618 upper=2.168 effort=100 velocity=5 -> lower=-2.6179 upper=2.6179 effort=100 velocity=5; origin xyz=0 0 0.123 rpy=0 0 0 -> xyz=0 0 0.123 rpy=0 0 -1.5708
- joint joint2: origin xyz=0 0 0 rpy=1.5708 -0.1359 -3.1416 -> xyz=0 0 0 rpy=1.5708 0 -1.5708
- joint joint3: limit lower=-2.967 upper=0 effort=100 velocity=5 -> lower=-2.967 upper=0 effort=100 velocity=3; origin xyz=0.28503 0 0 rpy=0 0 -1.7939 -> xyz=0.28358 0.028726 0 rpy=0 0 0.10095
- joint joint4: origin xyz=-0.021984 -0.25075 0 rpy=1.5708 0 0 -> xyz=-0.24221 0.068514 0 rpy=-1.5708 0 1.3826
- joint joint5: limit lower=-1.22 upper=1.22 effort=100 velocity=5 -> lower=-1.047 upper=1.047 effort=100 velocity=5; origin xyz=0 0 0 rpy=-1.5708 0 0 -> xyz=0 0 0 rpy=1.5708 0 0
- joint joint6: limit lower=-2.0944 upper=2.0944 effort=100 velocity=3 -> lower=-2.09439 upper=2.09439 effort=100 velocity=3; origin xyz=8.8259E-05 -0.091 0 rpy=1.5708 0 0 -> xyz=0 0.091 0.0014165 rpy=-1.5708 -3.1415926 0
- joint joint7: origin xyz=0 0 0.1358 rpy=1.5708 0 0 -> xyz=0 0 0.13503 rpy=1.5708 0 3.1415926; parent gripper_base -> link6
- joint joint8: origin xyz=0 0 0.1358 rpy=1.5708 0 -3.1416 -> xyz=0 0 0.13503 rpy=-1.5708 0 3.1415926; parent gripper_base -> link6
