Commit message: feat: Enhance Piper manipulator with improved joint synchronization and diagnostics
- Added immediate joint synchronization method in simulation to ensure accurate pose retrieval.
- Updated PiperHardware class to resolve end-effector link index dynamically and log diagnostics.
- Enhanced URDF structure to include TCP link for better kinematics handling.
- Improved forward kinematics to utilize immediate joint states for accurate position calculations.
- Added tests to verify correct behavior of movement commands and ensure no double offset in target positions.
- Refactored joint conversion methods to streamline motor unit calculations.

File: phosphobot/resources/urdf/piper/urdf/piper.urdf (robot description, URDF)
Before this commit: robot piper, 10 links, 9 joints
Links:
- added link tcp, mass 0.0001
Joints:
- added joint joint6_to_tcp: type fixed, parent link6, child tcp, origin xyz=0 0 0.14 rpy=0 0 0
